File: junior-computer/junior-computer.sch (KiCad schematic (older format))
At the start: 36 parts, among them IC1 6502, IC10 74LS01, IC2 2708, IC4 2114, IC5 2114, IC8 NE556, IC9 74LS00, Q1 1Mhz

Commit message: 'routing'
Connections:
- net +5V: now also S1.1 (A), S2.1 (A); no longer S1.2 (B), S2.2 (B)
- net A0: now also IC4.1 (A6), IC5.1 (A6); no longer IC4.5 (A0), IC5.5 (A0)
- net A1: now also IC4.2 (A5), IC5.2 (A5); no longer IC4.6 (A1), IC5.6 (A1)
- net A2: now also IC4.3 (A4), IC5.3 (A4); no longer IC4.7 (A2), IC5.7 (A2)
- net A3: now also IC4.17 (A7), IC5.17 (A7); no longer IC4.4 (A3), IC5.4 (A3)
- net A4: now also IC4.16 (A8), IC5.16 (A8); no longer IC4.3 (A4), IC5.3 (A4)
- net A5: now also IC4.5 (A0), IC5.5 (A0); no longer IC4.2 (A5), IC5.2 (A5)
- net A6: now also IC4.6 (A1), IC5.6 (A1); no longer IC4.1 (A6), IC5.1 (A6)
- net A7: now also IC4.7 (A2), IC5.7 (A2); no longer IC4.17 (A7), IC5.17 (A7)
- net A8: now also IC4.15 (A9), IC5.15 (A9); no longer IC4.16 (A8), IC5.16 (A8)
- net A9: now also IC4.4 (A3), IC5.4 (A3); no longer IC4.15 (A9), IC5.15 (A9)
- net at R17.2, R18.2: now also S1.2 (B); no longer S1.1 (A)
- net at R19.2, R20.2: now also S2.2 (B); no longer S2.1 (A)
Changed lines of the file:
@@
 K0
 Text Label 8600 1600 1    50   ~ 0
+A5
+Text Label 8700 1600 1    50   ~ 0
+A6
+Text Label 8800 1600 1    50   ~ 0
+A7
+Text Label 8900 1600 1    50   ~ 0
+A9
+Text Label 9000 1600 1    50   ~ 0
+A2
+Text Label 9100 1600 1    50   ~ 0
+A1
+Text Label 9200 1600 1    50   ~ 0
 A0
-Text Label 8700 1600 1    50   ~ 0
-A1
-Text Label 8800 1600 1    50   ~ 0
-A2
-Text Label 8900 1600 1    50   ~ 0
+Text Label 9300 1600 1    50   ~ 0
 A3
-Text Label 9000 1600 1    50   ~ 0
+Text Label 9400 1600 1    50   ~ 0
 A4
-Text Label 9100 1600 1    50   ~ 0
-A5
-Text Label 9200 1600 1    50   ~ 0
-A6
-Text Label 9300 1600 1    50   ~ 0
-A7
-Text Label 9400 1600 1    50   ~ 0
+Text Label 9500 1600 1    50   ~ 0
 A8
-Text Label 9500 1600 1    50   ~ 0
-A9
 Text Label 10100 3350 1    50   ~ 0
 RAM.RW
@@
 D7
 Text Label 8600 3350 1    50   ~ 0
+A5
+Text Label 8700 3350 1    50   ~ 0
+A6
+Text Label 8800 3350 1    50   ~ 0
+A7
+Text Label 8900 3350 1    50   ~ 0
+A9
+Text Label 9000 3350 1    50   ~ 0
+A2
+Text Label 9100 3350 1    50   ~ 0
+A1
+Text Label 9200 3350 1    50   ~ 0
 A0
-Text Label 8700 3350 1    50   ~ 0
-A1
-Text Label 8800 3350 1    50   ~ 0
-A2
-Text Label 8900 3350 1    50   ~ 0
+Text Label 9300 3350 1    50   ~ 0
 A3
-Text Label 9000 3350 1    50   ~ 0
+Text Label 9400 3350 1    50   ~ 0
 A4
-Text Label 9100 3350 1    50   ~ 0
-A5
-Text Label 9200 3350 1    50   ~ 0
-A6
-Text Label 9300 3350 1    50   ~ 0
-A7
-Text Label 9400 3350 1    50   ~ 0
+Text Label 9500 3350 1    50   ~ 0
 A8
-Text Label 9500 3350 1    50   ~ 0
-A9
 $Comp
 L Timer:NE556 IC8
@@
 F 3 "~" H 1050 6300 50  0001 C CNN
 	1    1050 6300
-	0    -1   -1   0
+	0    -1   1    0
 $EndComp
 $Comp
@@
 F 3 "~" H 3450 6300 50  0001 C CNN
 	1    3450 6300
-	0    -1   -1   0
-$EndComp
-$Comp
+	0    -1   1    0
+$EndComp
+$Comp

Commit message: routage complet
Parts:
- C12, C13: footprint elektor:CAP-POL-2 -> elektor:CAP-POL-1.5
Connections:
- net D0: now also IC4.11 (IO4); no longer IC4.14 (IO1)
- net D1: now also IC4.12 (IO3); no longer IC4.13 (IO2)
- net D2: now also IC4.13 (IO2); no longer IC4.12 (IO3)
- net D3: now also IC4.14 (IO1); no longer IC4.11 (IO4)
- net GNDD renamed GND
Changed lines of the file:
@@
 	9500 2750 9600 2650
 Text Label 9650 1600 1    50   ~ 0
+D3
+Text Label 9750 1600 1    50   ~ 0
+D2
+Text Label 9850 1600 1    50   ~ 0
+D1
+Text Label 9950 1600 1    50   ~ 0
 D0
-Text Label 9750 1600 1    50   ~ 0
-D1
-Text Label 9850 1600 1    50   ~ 0
-D2
-Text Label 9950 1600 1    50   ~ 0
-D3
 Text Label 10100 1600 1    50   ~ 0
 RAM.RW
@@
 F 0 "C12" H 6150 2800 50  0000 L CNN
 F 1 "1µ 16v" H 6000 2700 50  0000 L CNN
-F 2 "elektor:CAP-POL-2" H 6400 2750 50  0001 C CNN
+F 2 "elektor:CAP-POL-1.5" H 6400 2750 50  0001 C CNN
 F 3 "~" H 6400 2750 50  0001 C CNN
 	1    6400 2750
@@
 F 0 "C13" H 7050 2800 50  0000 L CNN
 F 1 "1µ 16v" H 6900 2700 50  0000 L CNN
-F 2 "elektor:CAP-POL-2" H 7300 2750 50  0001 C CNN
+F 2 "elektor:CAP-POL-1.5" H 7300 2750 50  0001 C CNN
 F 3 "~" H 7300 2750 50  0001 C CNN
 	1    7300 2750
@@
 $EndComp
 Wire Wire Line
-	7000 4100 7000 4250
-Wire Wire Line
-	7000 4450 7000 4600
+	7000 4100 7000 4150
+Wire Wire Line
+	7000 4450 7000 4550
 $Sheet
 S 9150 5200 1400 800
@@
 F1 "junior_computer_bus.sch" 50
 $EndSheet
+$Comp
+L power:VCC #PWR0156
+U 1 1 5F7B2451
+P 7250 4100
+F 0 "#PWR0156" H 7250 3950 50  0001 C CNN
+F 1 "VCC" H 7267 4273 50  0000 C CNN
+F 2 "" H 7250 4100 50  0001 C CNN
+F 3 "" H 7250 4100 50  0001 C CNN
+	1    7250 4100
+	1    0    0    -1
+$EndComp
+$Comp
+L power:GND #PWR0157
+U 1 1 5F7B299E
+P 7250 4600
+F 0 "#PWR0157" H 7250 4350 50  0001 C CNN
+F 1 "GND" H 7255 4427 50  0000 C CNN
+F 2 "" H 7250 4600 50  0001 C CNN
+F 3 "" H 7250 4600 50  0001 C CNN
+	1    7250 4600
+	1    0    0    -1
+$EndComp
+Wire Wire Line
+	7250 4100 7250 4150
+Wire Wire Line
+	7250 4150 7000 4150
+Connection ~ 7000 4150
+Wire Wire Line
+	7000 4150 7000 4250
+Wire Wire Line
+	7250 4600 7250 4550
+Wire Wire Line
+	7250 4550 7000 4550
 Wire Bus Line
 	8250 1100 10450 1100
@@
 Wire Bus Line
 	1500 900  8350 900
+Connection ~ 7000 4550
+Wire Wire Line
+	7000 4550 7000 4600
 $EndSCHEMATC

Commit message: amelioration dessin pistes
Parts:
- C8: footprint elektor:CAP-POL-2 -> elektor:CAP-POL-1.5
Changed lines of the file:
@@
 F 0 "C8" H 10700 2200 50  0000 L CNN
 F 1 "1µ 16v" H 10700 2100 50  0000 L CNN
-F 2 "elektor:CAP-POL-2" H 10550 2150 50  0001 C CNN
+F 2 "elektor:CAP-POL-1.5" H 10550 2150 50  0001 C CNN
 F 3 "~" H 10550 2150 50  0001 C CNN
 	1    10550 2150
