File: junior-computer/junior-computer.sch (KiCad schematic (older format))
At the start: 40 parts, among them IC1 6502, IC10 74LS01, IC2 2716, IC4 2114, IC5 2114, IC8 NE556, IC9 74LS00, J5 Conn_01x03_Female, Q1 1Mhz

Commit message: correction empreintes
Parts:
- C12: footprint elektor:CAP-2 -> elektor:CAP-2-HEX
Changed lines of the file:
@@
 F 0 "C12" V 1150 4750 50  0000 C CNN
 F 1 "470n" V 1450 4750 50  0000 C CNN
-F 2 "elektor:CAP-2" H 1338 4650 50  0001 C CNN
+F 2 "elektor:CAP-2-HEX" H 1338 4650 50  0001 C CNN
 F 3 "~" H 1300 4800 50  0001 C CNN
 	1    1300 4800
@@
 Wire Notes Line
 	5550 1200 5550 3500
+Wire Notes Line
+	5550 3500 8150 3500
 Wire Bus Line
 	8250 1100 10450 1100
@@
 Wire Bus Line
 	1500 900  8350 900
-Wire Notes Line
-	5550 3500 8150 3500
 $EndSCHEMATC
