File: junior-computer/junior-computer.sch (KiCad schematic (older format))
At the start: 40 parts, among them IC1 6502, IC10 74LS01, IC2 2716, IC4 2114, IC5 2114, IC8 NE556, IC9 74LS00, J5 Conn_01x03_Female, Q1 1Mhz

Commit message: finition platine
Parts:
- renumbered Q1 to X.Tal1
Changed lines of the file:
@@
 Connection ~ 1850 3000
 $Comp
-L Device:Crystal Q1
+L Device:Crystal X.Tal1
 U 1 1 5F71EF4A
 P 2750 3400
-F 0 "Q1" H 2750 3668 50  0000 C CNN
+F 0 "X.Tal1" H 2750 3668 50  0000 C CNN
 F 1 "1Mhz" H 2750 3577 50  0000 C CNN
 F 2 "elektor:Quartz" H 2750 3400 50  0001 C CNN
