File: junior-computer/junior-computer.kicad_pcb (KiCad board)
At the start: 2 copper layers, 217.2 x 113 mm, 86 parts, among them IC1 6502, IC10 74LS01, IC11 ULN2003, IC2 2716, IC3 6532, IC4 2114, IC5 2114, IC6 74LS145, IC7 74LS145, IC8 NE556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

Commit message: version commandée
Parts:
- removed the REF** at (40.6, 137.2)
- removed the REF** at (237.5, 33.0)
- removed the REF** at (237.5, 135.9)
- removed the REF** at (184.2, 88.9)
- added REF**: MountingHole_2.7mm_M2.5, Mounting_Holes:MountingHole_2.7mm_M2.5, F.Cu at (40.6, 137.2)
- added REF**: MountingHole_2.7mm_M2.5, Mounting_Holes:MountingHole_2.7mm_M2.5, F.Cu at (184.2, 88.9)
- added REF**: MountingHole_2.7mm_M2.5, Mounting_Holes:MountingHole_2.7mm_M2.5, F.Cu at (237.5, 33.0)
- added REF**: MountingHole_2.7mm_M2.5, Mounting_Holes:MountingHole_2.7mm_M2.5, F.Cu at (237.5, 135.9)
- turned C10 to 180 degrees
Connections:
- C10 pad 1: GND -> +5V
- C10 pad 2: +5V -> GND
Routing:
- net Net-(C1-Pad2): track 36.9 -> 40.7 mm
- net +5V: track 989.9 -> 992.6 mm
- net Net-(C1-Pad1): track 57.3 -> 55.0 mm
- net PB3: track 145.2 -> 146.1 mm
- net PB2: track 148.4 -> 148.9 mm
- net GND: track 1228.8 -> 1229.3 mm
Other:
- board text added: "Junior Computer Elektor 04/1980 | Replica @_Laurent_Fr_ 2020"

Commit message: junior interface update
Other:
- net class Default removed
