File: junior-computer/junior_computer_IO.sch (KiCad schematic (older format))
At the start: 39 parts, among them IC11 ULN2003, IC3 6532, IC6 74LS145, IC7 74LS145, J1 Display, J4 Conn_01x03_Female

Commit message: 'routing'
Parts:
- C7: footprint elektor:CAP-POL-2 -> elektor:CAP-POL-3
Changed lines of the file:
@@
 F 0 "C7" H 2400 4700 50  0000 C CNN
 F 1 "1µ 16V" H 2350 4600 50  0000 C CNN
-F 2 "elektor:CAP-POL-2" H 2600 4600 50  0001 C CNN
+F 2 "elektor:CAP-POL-3" H 2600 4600 50  0001 C CNN
 F 3 "~" H 2600 4600 50  0001 C CNN
 	1    2600 4600

Commit message: modifs schema
Connections:
- net +5V: now also C2.1
- net at R10.1, R11.1, R12.1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: no longer C2.1
Changed lines of the file:
@@
 $EndComp
-Wire Wire Line
-	6200 4950 6200 5050
-Connection ~ 6200 4950
 Wire Wire Line
 	6200 5250 6200 5300
@@
 Wire Wire Line
 	7450 2550 7450 2700
+Wire Wire Line
+	6200 5050 6750 5050
+Wire Wire Line
+	6750 5050 6750 5400
+Wire Wire Line
+	6750 5400 6900 5400
+Connection ~ 6900 5400
+Wire Notes Line
+	6100 5000 6850 5000
+Wire Notes Line
+	6850 5000 6850 5450
+Wire Notes Line
+	6850 5450 6100 5450
+Wire Notes Line
+	6100 5450 6100 5000
 Wire Bus Line
 	3000 3650 4550 3650

Commit message: version commandée
Connections:
- net +5V: now also C10.1; no longer C10.2
- net GNDD: now also C10.2; no longer C10.1
Changed lines of the file:
@@
 U 1 1 5F88FF29
 P 5000 2950
-F 0 "C10" V 4950 3250 50  0000 C CNN
-F 1 "1µ 16V" V 5050 3400 50  0000 C CNN
+F 0 "C10" V 4950 2650 50  0000 C CNN
+F 1 "1µ 16V" V 5050 2600 50  0000 C CNN
 F 2 "elektor:CAP-POL-2" H 5000 2950 50  0001 C CNN
 F 3 "~" H 5000 2950 50  0001 C CNN
 	1    5000 2950
-	0    1    1    0
+	0    -1   -1   0
 $EndComp
 $Comp
