File: junior-computer-display/junior-computer-display/junior-computer-display.kicad_pcb (KiCad board)
At the start: 2 copper layers, 77.5 x 31.8 mm, 11 parts, among them J1 Display

Commit message: lettrage
Routing:
- net Net-(Di6-Pad12): track 33.2 -> 31.9 mm
- net Net-(Di2-Pad12): track 76.3 -> 75.0 mm
- net Net-(Di4-Pad12): track 55.3 -> 54.1 mm
- net Net-(Di3-Pad12): track 65.8 -> 64.5 mm
- net Net-(Di1-Pad12): track 86.8 -> 85.5 mm
