File: junior-computer - original/junior-computer.sch (KiCad schematic (older format))
At the start: 40 parts, among them IC1 6502, IC10 74LS01, IC2 2716, IC4 2114, IC5 2114, IC8 NE556, IC9 74LS00, J5 Conn_01x03_Female, Q1 1Mhz

Commit message: modifs schema
Parts:
- removed C12: 470n, elektor:CAP-2, symbol Device:C
- removed D3: 1N4148, elektor:Diod-4, symbol Device:D
- removed unit 3 of IC10
- removed unit 4 of IC10
- removed unit 5 of IC10
- removed IC2: 2716, elektor:DIL-24, symbol junior_computer:2716
- removed unit 5 of IC9
- removed J5: Conn_01x03_Female, elektor:K4-K6, symbol Connector:Conn_01x03_Female
- removed R21, R22: 1k, elektor:Res-5, symbol Device:R
- removed R23: 820k, elektor:Res-5, symbol Device:R
- added C12, C13: 1µ 16v, elektor:CAP-POL-1.5, symbol Device:CP_Small
- added IC2: 2708, elektor:DIL-24, symbol junior_computer:2708
Connections:
- net labels added: +12V, -5V
- net labels removed: K4, K6
- wire segments 278 -> 258
Other:
- moved on the sheet: C14, C6
