File: junior-computer - original/junior_computer_IO.sch (KiCad schematic (older format))
At the start: 39 parts, among them IC11 ULN2003, IC3 6532, IC6 74LS145, IC7 74LS145, J1 Display, J4 Conn_01x03_Female

Commit message: modifs schema
Connections:
- net +5V: no longer C2.1
- net at R10.1, R11.1, R12.1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: now also C2.1
Changed lines of the file:
@@
 $EndComp
+Wire Wire Line
+	6200 4950 6200 5050
+Connection ~ 6200 4950
 Wire Wire Line
 	6200 5250 6200 5300
@@
 Wire Wire Line
 	7450 2550 7450 2700
-Wire Wire Line
-	6200 5050 6750 5050
-Wire Wire Line
-	6750 5050 6750 5400
-Wire Wire Line
-	6750 5400 6900 5400
 Wire Bus Line
 	3000 3650 4550 3650
@@
 Wire Bus Line
 	1700 3400 4550 3400
-Connection ~ 6900 5400
 $EndSCHEMATC
