File: ram-adapter/ram-adapter.kicad_pcb (KiCad board)
At the start: 2 copper layers, 33 x 33 mm, 5 parts, among them IC1 2114, IC2 6116, J1 Conn_01x04_Male, U1 74LS00

Commit message: version commandée
Parts:
- moved IC3 1.27 mm to (118.1, 59.7)
- renumbered U1 to IC3
Routing:
- net Net-(IC1-Pad10): track 25.4 -> 28.1 mm
- net Net-(IC2-Pad20): track 2.54 -> 3.81 mm
- net GND: track 32.2 -> 31.3 mm
- net VCC: track 43.1 -> 42.4 mm
Other:
- board size 33 x 33 mm -> 34.3 x 33 mm
- board text added: "2x2114->6116"
Changed lines of the file:
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@@
   (general
     (thickness 1.6)
-    (drawings 4)
-    (tracks 113)
+    (drawings 5)
+    (tracks 116)
     (zones 0)
     (modules 5)
@@
     (mod_text_size 1 1)
     (mod_text_width 0.15)
-    (pad_size 1.524 1.524)
-    (pad_drill 0.762)
+    (pad_size 1.7 1.7)
+    (pad_drill 0.8)
     (pad_to_mask_clearance 0.051)
     (solder_mask_min_width 0.25)
     (aux_axis_origin 0 0)
-    (visible_elements FFFFFF7F)
+    (visible_elements 7FFFFFFF)
     (pcbplotparams
       (layerselection 0x010fc_ffffffff)
@@
       (outputformat 1)
       (mirror false)
-      (drillshape 1)
+      (drillshape 0)
       (scaleselection 1)
-      (outputdirectory ""))
+      (outputdirectory "C:/Users/Laurent/Documents/kicad/junior-computer/ram-adapter/out/"))
   )
   (net 0 "")
@@
     (descr "24-lead though-hole mounted DIP package, row spacing 15.24 mm (600 mils)")
     (tags "THT DIP DIL PDIP 2.54mm 15.24mm 600mil")
-    (fp_text reference IC2 (at 17.78 -0.635) (layer F.SilkS)
+    (fp_text reference IC2 (at -2.54 -0.635) (layer F.SilkS)
       (effects (font (size 1 1) (thickness 0.15)))
     )
@@
     (descr "Through hole straight pin header, 1x04, 2.54mm pitch, single row")
     (tags "Through hole pin header THT 1x04 2.54mm single row")
-    (fp_text reference J1 (at 0 -2.33) (layer F.SilkS)
+    (fp_text reference J1 (at 0 -2.33) (layer F.SilkS) hide
       (effects (font (size 1 1) (thickness 0.15)))
     )
@@
     (fp_line (start 1.27 -1.27) (end 1.27 8.89) (layer F.Fab) (width 0.1))
     (fp_line (start -0.635 -1.27) (end 1.27 -1.27) (layer F.Fab) (width 0.1))
-    (pad 4 thru_hole oval (at 0 7.62 180) (size 1.7 1.7) (drill 1) (layers *.Cu *.Mask)
+    (pad 4 thru_hole oval (at 0 7.62 180) (size 1.7 1.7) (drill 0.8) (layers *.Cu *.Mask)
       (net 21 "Net-(IC2-Pad17)"))
-    (pad 3 thru_hole oval (at 0 5.08 180) (size 1.7 1.7) (drill 1) (layers *.Cu *.Mask)
+    (pad 3 thru_hole oval (at 0 5.08 180) (size 1.7 1.7) (drill 0.8) (layers *.Cu *.Mask)
       (net 22 "Net-(IC2-Pad16)"))
-    (pad 2 thru_hole oval (at 0 2.54 180) (size 1.7 1.7) (drill 1) (layers *.Cu *.Mask)
+    (pad 2 thru_hole oval (at 0 2.54 180) (size 1.7 1.7) (drill 0.8) (layers *.Cu *.Mask)
       (net 23 "Net-(IC2-Pad15)"))
-    (pad 1 thru_hole rect (at 0 0 180) (size 1.7 1.7) (drill 1) (layers *.Cu *.Mask)
+    (pad 1 thru_hole circle (at 0 0 180) (size 1.7 1.7) (drill 0.8) (layers *.Cu *.Mask)
       (net 24 "Net-(IC2-Pad14)"))
     (model ${KISYS3DMOD}/Pin_Headers.3dshapes/Pin_Header_Straight_1x04_Pitch2.54mm.wrl
@@
   )
   (module Housings_DIP:DIP-14_W7.62mm (layer F.Cu)
-    (at 116.84 59.69)
+    (at 118.11 59.69)
     (descr "14-lead though-hole mounted DIP package, row spacing 7.62 mm (300 mils)")
     (tags "THT DIP DIL PDIP 2.54mm 7.62mm 300mil")
-    (fp_text reference U1 (at 3.81 -2.33) (layer F.SilkS)
+    (fp_text reference IC3 (at 0 -2.54) (layer F.SilkS)
       (effects (font (size 1 1) (thickness 0.15)))
     )
@@
     )
   )
-  (gr_line (start 127 52.07) (end 127 85.09) (layer Edge.Cuts) (width 0.05))
-  (gr_line (start 93.98 52.07) (end 127 52.07) (layer Edge.Cuts) (width 0.05))
+  (gr_text 2x2114->6116 (at 121.92 54.61) (layer F.SilkS)
+    (effects (font (size 1 1) (thickness 0.2)))
+  )
+  (gr_line (start 128.27 52.07) (end 128.27 85.09) (layer Edge.Cuts) (width 0.05))
+  (gr_line (start 93.98 52.07) (end 128.27 52.07) (layer Edge.Cuts) (width 0.05))
   (gr_line (start 93.98 85.09) (end 93.98 52.07) (layer Edge.Cuts) (width 0.05))
-  (gr_line (start 127 85.09) (end 93.98 85.09) (layer Edge.Cuts) (width 0.05))
-  (segment (start 119.46 76.28) (end 119.46 80.01) (width 0.5) (layer B.Cu) (net 1))
-  (segment (start 116.84 74.93) (end 118.11 74.93) (width 0.5) (layer B.Cu) (net 1))
-  (segment (start 118.11 74.93) (end 119.46 76.28) (width 0.5) (layer B.Cu) (net 1))
+  (gr_line (start 128.27 85.09) (end 93.98 85.09) (layer Edge.Cuts) (width 0.05))
   (segment (start 101.6 81.28) (end 101.6 77.47) (width 0.5) (layer F.Cu) (net 1))
   (segment (start 99.06 82.55) (end 100.33 82.55) (width 0.5) (layer F.Cu) (net 1))
   (segment (start 100.33 82.55) (end 101.6 81.28) (width 0.5) (layer F.Cu) (net 1))
+  (segment (start 118.11 81.28) (end 101.6 81.28) (width 0.35) (layer F.Cu) (net 1))
   (segment (start 118.19 81.28) (end 119.46 80.01) (width 0.35) (layer F.Cu) (net 1))
   (segment (start 118.11 81.28) (end 118.19 81.28) (width 0.25) (layer F.Cu) (net 1))
-  (segment (start 118.11 81.28) (end 101.6 81.28) (width 0.35) (layer F.Cu) (net 1))
+  (segment (start 119.46 80.01) (end 119.46 75.645) (width 0.5) (layer F.Cu) (net 1))
+  (segment (start 119.46 75.645) (end 118.745 74.93) (width 0.5) (layer F.Cu) (net 1))
+  (segment (start 118.745 74.93) (end 118.11 74.93) (width 0.25) (layer F.Cu) (net 1))
   (segment (start 114.3 54.61) (end 111.76 54.61) (width 0.5) (layer B.Cu) (net 2))
   (segment (start 111.76 54.61) (end 109.22 57.15) (width 0.5) (layer B.Cu) (net 2))
-  (segment (start 119.38 54.61) (end 124.46 59.69) (width 0.5) (layer B.Cu) (net 2))
+  (segment (start 120.65 54.61) (end 125.73 59.69) (width 0.5) (layer B.Cu) (net 2))
   (segment (start 114.3 54.61) (end 119.38 54.61) (width 0.5) (layer B.Cu) (net 2))
-  (segment (start 121.92 60.325) (end 121.92 78.74) (width 0.5) (layer F.Cu) (net 2))
-  (segment (start 124.46 59.69) (end 122.555 59.69) (width 0.5) (layer F.Cu) (net 2))
-  (segment (start 122.555 59.69) (end 121.92 60.325) (width 0.5) (layer F.Cu) (net 2))
-  (segment (start 121.92 78.74) (end 121.92 79.375) (width 0.5) (layer F.Cu) (net 2))
-  (segment (start 122.555 80.01) (end 124.46 80.01) (width 0.5) (layer F.Cu) (net 2))
-  (segment (start 121.92 79.375) (end 122.555 80.01) (width 0.5) (layer F.Cu) (net 2))
+  (segment (start 123.19 60.325) (end 123.19 78.74) (width 0.5) (layer F.Cu) (net 2))
+  (segment (start 125.73 59.69) (end 123.825 59.69) (width 0.5) (layer F.Cu) (net 2))
+  (segment (start 123.825 59.69) (end 123.19 60.325) (width 0.5) (layer F.Cu) (net 2))
+  (segment (start 123.19 78.74) (end 123.19 79.375) (width 0.5) (layer F.Cu) (net 2))
+  (segment (start 123.19 79.375) (end 123.825 80.01) (width 0.5) (layer F.Cu) (net 2))
+  (segment (start 119.38 54.61) (end 120.65 54.61) (width 0.5) (layer B.Cu) (net 2))
   (segment (start 99.06 54.61) (end 102.87 54.61) (width 0.25) (layer B.Cu) (net 3))
   (segment (start 102.87 54.61) (end 107.95 59.69) (width 0.25) (layer B.Cu) (net 3))
@@
   (segment (start 107.95 74.93) (end 107.315 75.565) (width 0.25) (layer B.Cu) (net 15))
   (segment (start 101.6 59.69) (end 99.06 59.69) (width 0.25) (layer B.Cu) (net 16))
-  (segment (start 116.84 59.69) (end 116.84 62.23) (width 0.25) (layer B.Cu) (net 17))
+  (segment (start 118.11 59.69) (end 118.11 62.23) (width 0.25) (layer B.Cu) (net 17))
   (segment (start 109.22 77.47) (end 110.49 77.47) (width 0.25) (layer B.Cu) (net 17))
-  (segment (start 115.57 62.23) (end 115.57 74.93) (width 0.25) (layer B.Cu) (net 17))
   (segment (start 115.57 62.23) (end 114.3 62.23) (width 0.25) (layer B.Cu) (net 17))
   (segment (start 116.84 62.23) (end 115.57 62.23) (width 0.25) (layer B.Cu) (net 17))
-  (segment (start 115.57 75.325002) (end 114.695002 76.2) (width 0.25) (layer B.Cu) (net 17))
-  (segment (start 115.57 74.93) (end 115.57 75.325002) (width 0.25) (layer B.Cu) (net 17))
   (segment (start 114.695002 76.2) (end 111.76 76.2) (width 0.25) (layer B.Cu) (net 17))
   (segment (start 111.76 76.2) (end 110.49 77.47) (width 0.25) (layer B.Cu) (net 17))
+  (segment (start 114.695002 76.2) (end 115.57 76.2) (width 0.25) (layer B.Cu) (net 17))
+  (segment (start 115.57 76.2) (end 116.205 75.565) (width 0.25) (layer B.Cu) (net 17))
+  (segment (start 116.205 75.565) (end 116.205 62.23) (width 0.25) (layer B.Cu) (net 17))
+  (segment (start 116.205 62.23) (end 116.84 62.23) (width 0.25) (layer B.Cu) (net 17))
+  (segment (start 116.84 62.23) (end 118.11 62.23) (width 0.25) (layer B.Cu) (net 17))
   (segment (start 101.6 57.15) (end 99.06 57.15) (width 0.25) (layer B.Cu) (net 18))
   (segment (start 114.3 64.77) (end 116.84 64.77) (width 0.25) (layer F.Cu) (net 19))
+  (segment (start 116.84 64.77) (end 118.11 64.77) (width 0.25) (layer F.Cu) (net 19))
   (segment (start 96.52 67.31) (end 97.79 68.58) (width 0.25) (layer F.Cu) (net 21))
   (segment (start 97.79 68.58) (end 104.14 68.58) (width 0.25) (layer F.Cu) (net 21))
@@
   (segment (start 104.14 76.2) (end 107.95 80.01) (width 0.25) (layer F.Cu) (net 24))
   (segment (start 107.95 80.01) (end 114.3 80.01) (width 0.25) (layer F.Cu) (net 24))
-  (segment (start 124.46 62.23) (end 124.46 64.77) (width 0.25) (layer B.Cu) (net 25))
-  (segment (start 116.84 67.31) (end 116.84 69.85) (width 0.25) (layer B.Cu) (net 25))
-  (segment (start 124.46 64.77) (end 121.92 64.77) (width 0.25) (layer B.Cu) (net 25))
-  (segment (start 121.92 64.77) (end 120.65 66.04) (width 0.25) (layer B.Cu) (net 25))
-  (segment (start 120.65 66.04) (end 120.65 69.85) (width 0.25) (layer B.Cu) (net 25))
-  (segment (start 116.84 69.85) (end 120.65 69.85) (width 0.25) (layer B.Cu) (net 25))
-  (segment (start 120.65 69.85) (end 124.46 69.85) (width 0.25) (layer B.Cu) (net 25))
-  (segment (start 124.46 69.85) (end 124.46 72.39) (width 0.25) (layer B.Cu) (net 25))
+  (segment (start 125.73 62.23) (end 125.73 64.77) (width 0.25) (layer B.Cu) (net 25))
+  (segment (start 118.11 67.31) (end 118.11 69.85) (width 0.25) (layer B.Cu) (net 25))
+  (segment (start 125.73 64.77) (end 123.19 64.77) (width 0.25) (layer B.Cu) (net 25))
+  (segment (start 123.19 64.77) (end 121.92 66.04) (width 0.25) (layer B.Cu) (net 25))
+  (segment (start 121.92 66.04) (end 121.92 69.85) (width 0.25) (layer B.Cu) (net 25))
+  (segment (start 118.11 69.85) (end 121.92 69.85) (width 0.25) (layer B.Cu) (net 25))
+  (segment (start 121.92 69.85) (end 125.73 69.85) (width 0.25) (layer B.Cu) (net 25))
+  (segment (start 125.73 69.85) (end 125.73 72.39) (width 0.25) (layer B.Cu) (net 25))
 )
