File: junior-interface/junior-interface/junior-interface.sch (KiCad schematic (older format))
At the start: 24 parts, among them IC13 74LS27, IC14 74LS01, IC15 74LS30, IC16 74LS00, IC17 GAL16V8, IC2 2114, IC3 2114, IC4 2716, IC5 2716, J12 Conn_01x03_Male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

Commit message: junior interface update
Parts:
- IC2, IC3: symbol junior_computer:2114 -> junior-interface-rescue:2114-junior_computer
- IC4, IC5: symbol junior_computer:2716 -> junior-interface-rescue:2716-junior_computer
Changed lines of the file:
@@
 EESchema Schematic File Version 4
-LIBS:junior-interface-cache
 EELAYER 30 0
 EELAYER END
@@
 $EndDescr
 $Comp
-L junior_computer:2716 IC4
+L junior-interface-rescue:2716-junior_computer IC4
 U 1 1 5F92F96C
 P 1850 2000
@@
 $EndComp
 $Comp
-L junior_computer:2716 IC5
+L junior-interface-rescue:2716-junior_computer IC5
 U 1 1 5F93135B
 P 4300 2000
@@
 $EndSheet
 $Comp
-L junior_computer:2114 IC2
+L junior-interface-rescue:2114-junior_computer IC2
 U 1 1 5F934A67
 P 6750 2000
@@
 $EndComp
 $Comp
-L junior_computer:2114 IC3
+L junior-interface-rescue:2114-junior_computer IC3
 U 1 1 5F9351A2
 P 9250 2000
