File: junior-interface/junior-interface/junior_interface_busext.sch (KiCad schematic (older format))
At the start: 6 parts, among them IC10 74LS241, IC11 74LS243, IC12 74LS243, IC9 74LS241, J6 C64AC, J7 C64AB

Commit message: junior interface routage
Connections:
- net +5V: now also IC10.19 (OEb), IC9.19 (OEb)
- net AB0: now also J7.A26 (26A); no longer J7.B26 (26B)
- net AB1: now also J7.B26 (26B); no longer J7.A26 (26A)
- net AB10: now also J7.A21 (21A); no longer J7.B21 (21B)
- net AB11: now also J7.B21 (21B); no longer J7.A21 (21A)
- net AB12: now also J7.A20 (20A); no longer J7.B20 (20B)
- net AB13: now also J7.B20 (20B); no longer J7.A20 (20A)
- net AB14: now also J7.A19 (19A); no longer J7.B19 (19B)
- net AB15: now also J7.B19 (19B); no longer J7.A19 (19A)
- net AB2: now also J7.A25 (25A); no longer J7.B25 (25B)
- net AB3: now also J7.B25 (25B); no longer J7.A25 (25A)
- net AB4: now also J7.A24 (24A); no longer J7.B24 (24B)
- net AB5: now also J7.B24 (24B); no longer J7.A24 (24A)
- net AB6: now also J7.A23 (23A); no longer J7.B23 (23B)
- net AB7: now also J7.B23 (23B); no longer J7.A23 (23A)
- net AB8: now also J7.A22 (22A); no longer J7.B22 (22B)
- net AB9: now also J7.B22 (22B); no longer J7.A22 (22A)
- net GND: no longer IC10.19 (OEb), IC9.19 (OEb)
Changed lines of the file:
@@
 Text GLabel 2450 6500 2    50   Output ~ 0
 K2
-$Comp
-L power:GND #PWR0112
-U 1 1 5F9C054F
-P 2350 7200
-F 0 "#PWR0112" H 2350 6950 50  0001 C CNN
-F 1 "GND" V 2355 7072 50  0000 R CNN
-F 2 "" H 2350 7200 50  0001 C CNN
-F 3 "" H 2350 7200 50  0001 C CNN
-	1    2350 7200
-	0    -1   -1   0
-$EndComp
 Wire Wire Line
 	1550 6200 2050 6200
@@
 	6150 6050 6050 6050
 Wire Wire Line
-	6050 6050 6050 6150
-Wire Wire Line
-	6150 6150 6050 6150
-Connection ~ 6050 6150
-Wire Wire Line
-	6050 6150 6050 6250
-Wire Wire Line
 	6150 4100 6050 4100
-Wire Wire Line
-	6050 4100 6050 4200
-Wire Wire Line
-	6150 4200 6050 4200
-Connection ~ 6050 4200
-Wire Wire Line
-	6050 4200 6050 4350
 Wire Bus Line
 	5450 650  9550 650
@@
 DB6
 Text Label 2650 4600 0    50   ~ 0
+AB14
+Text Label 2650 4700 0    50   ~ 0
 AB15
-Text Label 2650 4700 0    50   ~ 0
-AB14
 Text Label 2650 4800 0    50   ~ 0
+AB12
+Text Label 2650 4900 0    50   ~ 0
 AB13
-Text Label 2650 4900 0    50   ~ 0
-AB12
 Text Label 2650 5000 0    50   ~ 0
+AB10
+Text Label 2650 5100 0    50   ~ 0
 AB11
-Text Label 2650 5100 0    50   ~ 0
-AB10
 Text Label 2650 5200 0    50   ~ 0
+AB8
+Text Label 2650 5300 0    50   ~ 0
 AB9
-Text Label 2650 5300 0    50   ~ 0
-AB8
 Text Label 2650 5400 0    50   ~ 0
+AB6
+Text Label 2650 5500 0    50   ~ 0
 AB7
-Text Label 2650 5500 0    50   ~ 0
-AB6
 Text Label 2650 5600 0    50   ~ 0
+AB4
+Text Label 2650 5700 0    50   ~ 0
 AB5
-Text Label 2650 5700 0    50   ~ 0
-AB4
 Text Label 2650 5800 0    50   ~ 0
+AB2
+Text Label 2650 5900 0    50   ~ 0
 AB3
-Text Label 2650 5900 0    50   ~ 0
-AB2
 Text Label 2650 6000 0    50   ~ 0
+AB0
+Text Label 2650 6100 0    50   ~ 0
 AB1
-Text Label 2650 6100 0    50   ~ 0
-AB0
 Text GLabel 3000 1300 1    50   BiDi ~ 0
 DB[0..7]
@@
 Text Label 3250 1800 1    50   ~ 0
 AB[0..15]
+Wire Wire Line
+	6050 4100 6050 4350
+Wire Wire Line
+	6050 6050 6050 6250
+$Comp
+L power:+5V #PWR0183
+U 1 1 5F98E2EF
+P 6000 6150
+F 0 "#PWR0183" H 6000 6000 50  0001 C CNN
+F 1 "+5V" H 6015 6323 50  0000 C CNN
+F 2 "" H 6000 6150 50  0001 C CNN
+F 3 "" H 6000 6150 50  0001 C CNN
+	1    6000 6150
+	0    -1   -1   0
+$EndComp
+$Comp
+L power:+5V #PWR0184
+U 1 1 5F98E8A0
+P 6000 4200
+F 0 "#PWR0184" H 6000 4050 50  0001 C CNN
+F 1 "+5V" H 6015 4373 50  0000 C CNN
+F 2 "" H 6000 4200 50  0001 C CNN
+F 3 "" H 6000 4200 50  0001 C CNN
+	1    6000 4200
+	0    -1   -1   0
+$EndComp
+Wire Wire Line
+	6150 4200 6000 4200
+Wire Wire Line
+	6150 6150 6000 6150
 Wire Bus Line
 	3250 1300 3250 7350

Commit message: junior interface routage
Connections:
- net +12V: now also J7.A17 (17A); no longer J7.B17 (17B)
- net -5V: now also J7.B18 (18B); no longer J7.A18 (18A)
- net DB0: now also J7.A7 (7A); no longer J7.B7 (7B)
- net DB1: now also J7.B7 (7B); no longer J7.A7 (7A)
- net DB2: now also J7.A8 (8A); no longer J7.B8 (8B)
- net DB3: now also J7.B8 (8B); no longer J7.A8 (8A)
- net DB4: now also J7.A9 (9A); no longer J7.B9 (9B)
- net DB5: now also J7.B9 (9B); no longer J7.A9 (9A)
- net DB6: now also J7.A10 (10A); no longer J7.B10 (10B)
- net DB7: now also J7.B10 (10B); no longer J7.A10 (10A)
- net EX: now also J7.A30 (30A); no longer J7.B30 (30B)
- net IRQ: now also J7.B12 (12B); no longer J7.A12 (12A)
- net K1: now also J7.B29 (29B); no longer J7.A29 (29A)
- net K2: now also J7.A28 (28A); no longer J7.B28 (28B)
- net K3: now also J7.A18 (18A); no longer J7.B18 (18B)
- net K4: now also J7.B17 (17B); no longer J7.A17 (17A)
- net K5: now also J7.B15 (15B); no longer J7.A15 (15A)
- net K6: now also J7.A15 (15A); no longer J7.B15 (15B)
- net K7: now also J7.B14 (14B); no longer J7.A14 (14A)
- net NMI: now also J7.A12 (12A); no longer J7.B12 (12B)
- net PHI1: now also J7.B30 (30B); no longer J7.A30 (30A)
- net PHI2: now also J7.B27 (27B); no longer J7.A27 (27A)
- net RAM.RW: now also J7.B31 (31B); no longer J7.A31 (31A)
- net RDY: now also J7.A5 (5A); no longer J7.B5 (5B)
- net RES: now also J7.B5 (5B); no longer J7.A5 (5A)
- net RW: now also J7.A29 (29A); no longer J7.B29 (29B)
- net SO: now also J7.A14 (14A); no longer J7.B14 (14B)
Changed lines of the file:
@@
 L power:+12V #PWR0108
 U 1 1 5F98F62B
-P 1750 4300
-F 0 "#PWR0108" H 1750 4150 50  0001 C CNN
-F 1 "+12V" V 1765 4428 50  0000 L CNN
-F 2 "" H 1750 4300 50  0001 C CNN
-F 3 "" H 1750 4300 50  0001 C CNN
-	1    1750 4300
+P 2050 4200
+F 0 "#PWR0108" H 2050 4050 50  0001 C CNN
+F 1 "+12V" V 2065 4328 50  0000 L CNN
+F 2 "" H 2050 4200 50  0001 C CNN
+F 3 "" H 2050 4200 50  0001 C CNN
+	1    2050 4200
 	0    1    1    0
 $EndComp
@@
 L power:-5V #PWR0109
 U 1 1 5F992A76
-P 1750 4400
-F 0 "#PWR0109" H 1750 4500 50  0001 C CNN
-F 1 "-5V" V 1765 4528 50  0000 L CNN
-F 2 "" H 1750 4400 50  0001 C CNN
-F 3 "" H 1750 4400 50  0001 C CNN
-	1    1750 4400
+P 2050 4500
+F 0 "#PWR0109" H 2050 4600 50  0001 C CNN
+F 1 "-5V" V 2065 4628 50  0000 L CNN
+F 2 "" H 2050 4500 50  0001 C CNN
+F 3 "" H 2050 4500 50  0001 C CNN
+	1    2050 4500
 	0    1    1    0
 $EndComp
@@
 	0    -1   -1   0
 $EndComp
+Text GLabel 2300 1900 2    50   Output ~ 0
+RES
 Text GLabel 2050 1800 2    50   Output ~ 0
-RES
-Text GLabel 2300 1900 2    50   Output ~ 0
 RDY
 Wire Wire Line
@@
 Wire Wire Line
 	2300 1900 1550 1900
+Text GLabel 2050 3200 2    50   Output ~ 0
+NMI
 Text GLabel 2450 3300 2    50   Output ~ 0
-NMI
-Text GLabel 2050 3200 2    50   Output ~ 0
 IRQ
-Text GLabel 2050 4200 2    50   Output ~ 0
+Text GLabel 1750 4300 2    50   Output ~ 0
 K4
+Text GLabel 2450 3900 2    50   Output ~ 0
+K5
 Text GLabel 2050 3800 2    50   Output ~ 0
-K5
-Text GLabel 2450 3900 2    50   Output ~ 0
 K6
+Text GLabel 2450 3700 2    50   Output ~ 0
+K7
 Text GLabel 2050 3600 2    50   Output ~ 0
-K7
-Text GLabel 2450 3700 2    50   Output ~ 0
 SO
 Wire Wire Line
@@
 Wire Wire Line
 	1550 4200 2050 4200
-Text GLabel 2050 4500 2    50   Output ~ 0
+Text GLabel 1750 4400 2    50   Output ~ 0
 K3
 Wire Wire Line
 	2050 4500 1550 4500
+Text GLabel 2050 6600 2    50   Output ~ 0
+RW
+Text GLabel 2050 7100 2    50   Output ~ 0
+RAM.RW
+Text GLabel 2450 6900 2    50   Output ~ 0
+PHI1
+Text GLabel 2050 6300 2    50   Output ~ 0
+PHI2
+Text GLabel 2050 6800 2    50   Output ~ 0
+EX
 Text GLabel 2450 6700 2    50   Output ~ 0
-RW
-Text GLabel 2050 7000 2    50   Output ~ 0
-RAM.RW
-Text GLabel 2050 6800 2    50   Output ~ 0
-PHI1
-Text GLabel 2050 6200 2    50   Output ~ 0
-PHI2
-Text GLabel 2450 6900 2    50   Output ~ 0
-EX
-Text GLabel 2050 6600 2    50   Output ~ 0
 K1
-Text GLabel 2450 6500 2    50   Output ~ 0
+Text GLabel 2450 6400 2    50   Output ~ 0
 K2
 Wire Wire Line
-	1550 6200 2050 6200
-Wire Wire Line
-	1550 6500 2450 6500
-Wire Wire Line
 	1550 6600 2050 6600
 Wire Wire Line
@@
 Wire Wire Line
 	1550 6900 2450 6900
-Wire Wire Line
-	1550 7000 2050 7000
 Entry Wire Line
 	5450 5950 5550 5850
@@
 	1550 6100 2900 6100
 Text Label 2700 2200 0    50   ~ 0
+DB0
+Text Label 2700 2300 0    50   ~ 0
 DB1
-Text Label 2700 2300 0    50   ~ 0
-DB0
 Text Label 2700 2400 0    50   ~ 0
+DB2
+Text Label 2700 2500 0    50   ~ 0
 DB3
-Text Label 2700 2500 0    50   ~ 0
-DB2
 Text Label 2700 2600 0    50   ~ 0
+DB4
+Text Label 2700 2700 0    50   ~ 0
 DB5
-Text Label 2700 2700 0    50   ~ 0
-DB4
 Text Label 2700 2800 0    50   ~ 0
+DB6
+Text Label 2700 2900 0    50   ~ 0
 DB7
-Text Label 2700 2900 0    50   ~ 0
-DB6
 Text Label 2650 4600 0    50   ~ 0
 AB14
@@
 Wire Wire Line
 	6150 6150 6000 6150
+Wire Wire Line
+	2050 6300 1550 6300
+Wire Wire Line
+	2450 6400 1550 6400
+Wire Wire Line
+	2050 7100 1550 7100
 Wire Bus Line
 	3250 1300 3250 7350

Commit message: junior interface routage
Connections:
- net GND: now also J6.A16 (16A), J6.C16 (16C)
Changed lines of the file:
@@
 Wire Wire Line
 	2050 7100 1550 7100
+$Comp
+L power:GND #PWR0192
+U 1 1 5FA4AAE0
+P 4750 4050
+F 0 "#PWR0192" H 4750 3800 50  0001 C CNN
+F 1 "GND" H 4755 3877 50  0000 C CNN
+F 2 "" H 4750 4050 50  0001 C CNN
+F 3 "" H 4750 4050 50  0001 C CNN
+	1    4750 4050
+	0    -1   -1   0
+$EndComp
+Wire Wire Line
+	4650 4050 4650 4000
+Wire Wire Line
+	4650 4000 4450 4000
+Wire Wire Line
+	4650 4050 4750 4050
+Wire Wire Line
+	4450 4100 4650 4100
+Wire Wire Line
+	4650 4100 4650 4050
 Wire Bus Line
 	3250 1300 3250 7350
@@
 Wire Bus Line
 	5450 650  5450 7400
+Connection ~ 4650 4050
 $EndSCHEMATC

Commit message: junior interface routage
Connections:
- net EX: no longer J7.A30 (30A)
- net K1: no longer J7.B29 (29B)
- net K2: no longer J7.A28 (28A)
- net K3: no longer J7.A18 (18A)
- net K4: no longer J7.B17 (17B)
- net K5: no longer J7.B15 (15B)
- net K6: no longer J7.A15 (15A)
- net K7: no longer J7.B14 (14B)
Changed lines of the file:
@@
 	0    1    1    0
 $EndComp
-Wire Wire Line
-	1750 4300 1550 4300
 $Comp
 L power:-5V #PWR0109
@@
 	0    1    1    0
 $EndComp
-Wire Wire Line
-	1750 4400 1550 4400
 $Comp
 L power:GND #PWR0110
@@
 Text GLabel 2450 3300 2    50   Output ~ 0
 IRQ
-Text GLabel 1750 4300 2    50   Output ~ 0
-K4
-Text GLabel 2450 3900 2    50   Output ~ 0
-K5
-Text GLabel 2050 3800 2    50   Output ~ 0
-K6
-Text GLabel 2450 3700 2    50   Output ~ 0
-K7
 Text GLabel 2050 3600 2    50   Output ~ 0
 SO
@@
 	1550 3600 2050 3600
 Wire Wire Line
-	1550 3700 2450 3700
-Wire Wire Line
-	1550 3800 2050 3800
-Wire Wire Line
-	1550 3900 2450 3900
-Wire Wire Line
 	1550 4200 2050 4200
-Text GLabel 1750 4400 2    50   Output ~ 0
-K3
 Wire Wire Line
 	2050 4500 1550 4500
@@
 Text GLabel 2050 6300 2    50   Output ~ 0
 PHI2
-Text GLabel 2050 6800 2    50   Output ~ 0
-EX
-Text GLabel 2450 6700 2    50   Output ~ 0
-K1
-Text GLabel 2450 6400 2    50   Output ~ 0
-K2
 Wire Wire Line
 	1550 6600 2050 6600
-Wire Wire Line
-	1550 6700 2450 6700
-Wire Wire Line
-	1550 6800 2050 6800
 Wire Wire Line
 	1550 6900 2450 6900
@@
 	2050 6300 1550 6300
 Wire Wire Line
-	2450 6400 1550 6400
-Wire Wire Line
 	2050 7100 1550 7100
 $Comp
@@
 Wire Wire Line
 	4650 4100 4650 4050
+Connection ~ 4650 4050
 Wire Bus Line
 	3250 1300 3250 7350
@@
 Wire Bus Line
 	5450 650  5450 7400
-Connection ~ 4650 4050
 $EndSCHEMATC
