File: junior-interface/junior-interface/juniour_interface_out.sch (KiCad schematic (older format))
At the start: 68 parts, among them IC14 74LS01, IC6 NE565, IC7 LM311, IC8 LM311, J1 Output, J10 DB25_Female, J2 Output, J24 P, J25 Q, J26 D4, J27 , J28 D5, J29 Conn_01x06_Male, J4 Output, J9 Output, P1 5k, P2 1k, T1 BC547, T2 BC516, T3 BC516

Commit message: junior bus
Parts:
- J10: footprint Connectors_DSub:DSUB-25_Female_Horizontal_Pitch2.77x2.84mm_EdgePinOffset9.90mm_Housed_MountingHolesOffset11.32mm -> elektor:DB25-F-CI
- P2: footprint Potentiometers:Potentiometer_Trimmer_ACP_CA9v_Horizontal_Px10.0mm_Py5.0mm -> elektor:POT
- T1, T2, T3: footprint TO_SOT_Packages_THT:TO-92_Molded_Wide -> elektor:TO-92
Changed lines of the file:
@@
 F 0 "J10" H 4680 4996 50  0000 L CNN
 F 1 "DB25_Female" H 4680 4905 50  0000 L CNN
-F 2 "Connectors_DSub:DSUB-25_Female_Horizontal_Pitch2.77x2.84mm_EdgePinOffset9.90mm_Housed_MountingHolesOffset11.32mm" H 4500 4950 50  0001 C CNN
+F 2 "elektor:DB25-F-CI" H 4500 4950 50  0001 C CNN
 F 3 " ~" H 4500 4950 50  0001 C CNN
 	1    4500 4950
@@
 F 0 "T1" H 1991 4796 50  0000 L CNN
 F 1 "BC547" H 1991 4705 50  0000 L CNN
-F 2 "TO_SOT_Packages_THT:TO-92_Molded_Wide" H 2000 4675 50  0001 L CIN
+F 2 "elektor:TO-92" H 2000 4675 50  0001 L CIN
 F 3 "http://www.fairchildsemi.com/ds/BC/BC547.pdf" H 1800 4750 50  0001 L CNN
 	1    1800 4750
@@
 F 0 "T2" H 6791 4804 50  0000 L CNN
 F 1 "BC516" H 6791 4895 50  0000 L CNN
-F 2 "TO_SOT_Packages_THT:TO-92_Molded_Wide" H 6800 4775 50  0001 L CIN
+F 2 "elektor:TO-92" H 6800 4775 50  0001 L CIN
 F 3 "http://www.fairchildsemi.com/ds/BC/BC516.pdf" H 6600 4850 50  0001 L CNN
 	1    6600 4850
@@
 F 0 "T3" H 9591 4804 50  0000 L CNN
 F 1 "BC516" H 9591 4895 50  0000 L CNN
-F 2 "TO_SOT_Packages_THT:TO-92_Molded_Wide" H 9600 4775 50  0001 L CIN
+F 2 "elektor:TO-92" H 9600 4775 50  0001 L CIN
 F 3 "http://www.fairchildsemi.com/ds/BC/BC516.pdf" H 9400 4850 50  0001 L CNN
 	1    9400 4850
@@
 F 0 "P2" H 2980 3246 50  0000 R CNN
 F 1 "1k" H 2980 3155 50  0000 R CNN
-F 2 "Potentiometers:Potentiometer_Trimmer_ACP_CA9v_Horizontal_Px10.0mm_Py5.0mm" H 3050 3200 50  0001 C CNN
+F 2 "elektor:POT" H 3050 3200 50  0001 C CNN
 F 3 "~" H 3050 3200 50  0001 C CNN
 	1    3050 3200

Commit message: junior interface update
Parts:
- IC6: symbol junior_computer:NE565 -> junior-interface-rescue:NE565-junior_computer
- IC7, IC8: symbol Comparator:LM311 -> junior-interface-rescue:LM311-Comparator
- Re1, Re2: symbol junior_computer:relay_reed -> junior-interface-rescue:relay_reed-junior_computer
- renumbered J4 to J3, J9 to J4
Changed lines of the file:
@@
 EESchema Schematic File Version 4
-LIBS:junior-interface-cache
 EELAYER 30 0
 EELAYER END
@@
 $EndDescr
 $Comp
-L Comparator:LM311 IC7
+L junior-interface-rescue:LM311-Comparator IC7
 U 1 1 5F93A9A0
 P 3500 1600
+AR Path="/5F93A9A0" Ref="IC7"  Part="1"
+AR Path="/5F939FEF/5F93A9A0" Ref="IC7"  Part="1"
 F 0 "IC7" H 3844 1646 50  0000 L CNN
 F 1 "LM311" H 3844 1555 50  0000 L CNN
@@
 $EndComp
 $Comp
-L Comparator:LM311 IC8
+L junior-interface-rescue:LM311-Comparator IC8
 U 1 1 5F93AFD8
 P 3200 6350
+AR Path="/5F93AFD8" Ref="IC8"  Part="1"
+AR Path="/5F939FEF/5F93AFD8" Ref="IC8"  Part="1"
 F 0 "IC8" H 3300 6250 50  0000 L CNN
 F 1 "LM311" H 3300 6150 50  0000 L CNN
@@
 $EndComp
 $Comp
-L junior_computer:NE565 IC6
+L junior-interface-rescue:NE565-junior_computer IC6
 U 1 1 5F952C6E
 P 6850 1300
@@
 $EndComp
 $Comp
-L junior_computer:relay_reed Re1
+L junior-interface-rescue:relay_reed-junior_computer Re1
 U 1 1 5F9A7987
 P 6900 5500
@@
 $EndComp
 $Comp
-L Connector:Conn_01x02_Female J4
+L Connector:Conn_01x02_Female J3
 U 1 1 5F9A972A
 P 7950 5450
-F 0 "J4" H 7978 5426 50  0000 L CNN
+F 0 "J3" H 7978 5426 50  0000 L CNN
 F 1 "Output" H 7978 5335 50  0000 L CNN
 F 2 "elektor:RCA_CI_1" H 7950 5450 50  0001 C CNN
@@
 $EndComp
 $Comp
-L junior_computer:relay_reed Re2
+L junior-interface-rescue:relay_reed-junior_computer Re2
 U 1 1 5F9C15C0
 P 9700 5500
@@
 $EndComp
 $Comp
-L Connector:Conn_01x02_Female J9
+L Connector:Conn_01x02_Female J4
 U 1 1 5F9C15D4
 P 10750 5450
-F 0 "J9" H 10778 5426 50  0000 L CNN
+F 0 "J4" H 10778 5426 50  0000 L CNN
 F 1 "Output" H 10778 5335 50  0000 L CNN
 F 2 "elektor:RCA_CI_1" H 10750 5450 50  0001 C CNN
