File: junior-internal-bus/junior-internal-bus/junior-internal-bus.sch (KiCad schematic (older format))
At the start: 3 parts, among them J1 C64AC, J2 C64AC, J3 Conn_01x06_Male

Commit message: junior bus
Parts:
- removed J3: Conn_01x06_Male, Connectors_Molex:Molex_MiniFit-JR-5569-06A2_2x03x4.20mm_Angled, symbol Connector:Conn_01x06_Male
Connections:
- net +12V: no longer names the net of J1.C17 (17C), J2.C17 (17C)
- net +5V: no longer names the net of J1.A1 (1A), J1.C1 (1C), J2.A1 (1A), J2.C1 (1C)
- net -12V: no longer names the net of J1.C2 (2C), J2.C2 (2C)
- net -5V: no longer names the net of J1.A18 (18A), J2.A18 (18A)
Changed lines of the file:
@@
 EESchema Schematic File Version 4
+LIBS:junior-internal-bus-cache
 EELAYER 30 0
 EELAYER END
@@
 	5550 3300 5550 4600
 Wire Wire Line
-	5650 4600 5650 3950
-Wire Wire Line
-	5750 3300 5750 3850
-Wire Wire Line
 	5850 3300 5850 4600
 Wire Wire Line
@@
 Wire Wire Line
 	8650 4600 8650 3300
-Wire Wire Line
-	8750 3300 8750 4050
 Wire Wire Line
 	8950 3300 8950 3750
@@
 Wire Wire Line
 	2750 4400 2750 3300
-$Comp
-L power:GND #PWR0101
-U 1 1 5F900CB0
-P 9450 4500
-F 0 "#PWR0101" H 9450 4250 50  0001 C CNN
-F 1 "GND" H 9455 4327 50  0000 C CNN
-F 2 "" H 9450 4500 50  0001 C CNN
-F 3 "" H 9450 4500 50  0001 C CNN
-	1    9450 4500
-	1    0    0    -1
-$EndComp
 $Comp
 L power:GND #PWR0102
@@
 	2350 4400 2350 4650
 Wire Wire Line
-	9450 4400 9450 4500
-$Comp
-L power:GND #PWR0103
-U 1 1 5F9091E2
-P 4250 6400
-F 0 "#PWR0103" H 4250 6150 50  0001 C CNN
-F 1 "GND" H 4255 6227 50  0000 C CNN
-F 2 "" H 4250 6400 50  0001 C CNN
-F 3 "" H 4250 6400 50  0001 C CNN
-	1    4250 6400
-	1    0    0    -1
-$EndComp
-$Comp
-L power:+5V #PWR0104
-U 1 1 5F9097C5
-P 4600 5650
-F 0 "#PWR0104" H 4600 5500 50  0001 C CNN
-F 1 "+5V" H 4615 5823 50  0000 C CNN
-F 2 "" H 4600 5650 50  0001 C CNN
-F 3 "" H 4600 5650 50  0001 C CNN
-	1    4600 5650
-	1    0    0    -1
-$EndComp
-$Comp
-L power:-12V #PWR0105
-U 1 1 5F909B0D
-P 5150 5650
-F 0 "#PWR0105" H 5150 5750 50  0001 C CNN
-F 1 "-12V" H 5165 5823 50  0000 C CNN
-F 2 "" H 5150 5650 50  0001 C CNN
-F 3 "" H 5150 5650 50  0001 C CNN
-	1    5150 5650
-	1    0    0    -1
-$EndComp
-$Comp
-L power:+12V #PWR0106
-U 1 1 5F90A1E0
-P 5400 5650
-F 0 "#PWR0106" H 5400 5500 50  0001 C CNN
-F 1 "+12V" H 5415 5823 50  0000 C CNN
-F 2 "" H 5400 5650 50  0001 C CNN
-F 3 "" H 5400 5650 50  0001 C CNN
-	1    5400 5650
-	1    0    0    -1
-$EndComp
-$Comp
-L power:-5V #PWR0107
-U 1 1 5F90B100
-P 4850 5650
-F 0 "#PWR0107" H 4850 5750 50  0001 C CNN
-F 1 "-5V" H 4865 5823 50  0000 C CNN
-F 2 "" H 4850 5650 50  0001 C CNN
-F 3 "" H 4850 5650 50  0001 C CNN
-	1    4850 5650
-	1    0    0    -1
-$EndComp
-Wire Wire Line
-	4000 5800 4250 5800
-Wire Wire Line
-	4250 5800 4250 6100
-Wire Wire Line
-	4000 6100 4250 6100
-Connection ~ 4250 6100
-Wire Wire Line
-	4250 6100 4250 6400
-Wire Wire Line
-	4000 6200 4600 6200
-Wire Wire Line
-	4600 6200 4600 5650
-$Comp
-L Connector:Conn_01x06_Male J3
-U 1 1 5F9125F6
-P 3800 6000
-F 0 "J3" H 3908 6381 50  0000 C CNN
-F 1 "Conn_01x06_Male" H 3908 6290 50  0000 C CNN
-F 2 "Connectors_Molex:Molex_MiniFit-JR-5569-06A2_2x03x4.20mm_Angled" H 3800 6000 50  0001 C CNN
-F 3 "~" H 3800 6000 50  0001 C CNN
-	1    3800 6000
-	1    0    0    -1
-$EndComp
-Wire Wire Line
-	4000 6300 5150 6300
-Wire Wire Line
-	5150 6300 5150 5650
-Wire Wire Line
-	4000 5900 4850 5900
-Wire Wire Line
-	4850 5900 4850 5650
-Wire Wire Line
-	4000 6000 5400 6000
-Wire Wire Line
-	5400 6000 5400 5650
-$Comp
-L power:+5V #PWR0108
-U 1 1 5F91B534
-P 9450 3650
-F 0 "#PWR0108" H 9450 3500 50  0001 C CNN
-F 1 "+5V" H 9465 3823 50  0000 C CNN
-F 2 "" H 9450 3650 50  0001 C CNN
-F 3 "" H 9450 3650 50  0001 C CNN
-	1    9450 3650
-	1    0    0    -1
-$EndComp
-Wire Wire Line
 	8950 3750 9050 3750
 Connection ~ 8950 3750
@@
 	9050 3750 9050 3300
 Wire Wire Line
-	9050 3750 9450 3750
-Wire Wire Line
-	9450 3750 9450 3650
-Wire Wire Line
 	9050 3750 9050 4600
 Wire Wire Line
 	8950 3750 8950 4600
 Wire Wire Line
-	8450 4400 9450 4400
-$Comp
-L power:+12V #PWR0109
-U 1 1 5F924BF8
-P 9750 3650
-F 0 "#PWR0109" H 9750 3500 50  0001 C CNN
-F 1 "+12V" H 9765 3823 50  0000 C CNN
-F 2 "" H 9750 3650 50  0001 C CNN
-F 3 "" H 9750 3650 50  0001 C CNN
-	1    9750 3650
+	8850 3300 8850 4600
+Wire Wire Line
+	5750 3300 5750 4600
+Wire Wire Line
+	5650 3300 5650 4600
+Wire Wire Line
+	8750 3300 8750 4600
+$Comp
+L power:GND #PWR?
+U 1 1 5FA0E4D1
+P 9550 4600
+F 0 "#PWR?" H 9550 4350 50  0001 C CNN
+F 1 "GND" H 9555 4427 50  0000 C CNN
+F 2 "" H 9550 4600 50  0001 C CNN
+F 3 "" H 9550 4600 50  0001 C CNN
+	1    9550 4600
 	1    0    0    -1
 $EndComp
-$Comp
-L power:-5V #PWR0110
-U 1 1 5F924FBF
-P 10050 3650
-F 0 "#PWR0110" H 10050 3750 50  0001 C CNN
-F 1 "-5V" H 10065 3823 50  0000 C CNN
-F 2 "" H 10050 3650 50  0001 C CNN
-F 3 "" H 10050 3650 50  0001 C CNN
-	1    10050 3650
-	1    0    0    -1
-$EndComp
-Wire Wire Line
-	5750 3850 9750 3850
-Wire Wire Line
-	9750 3850 9750 3650
-Connection ~ 5750 3850
-Wire Wire Line
-	5750 3850 5750 4600
-Wire Wire Line
-	5650 3950 10050 3950
-Wire Wire Line
-	10050 3950 10050 3650
-Connection ~ 5650 3950
-Wire Wire Line
-	5650 3950 5650 3300
-$Comp
-L power:-12V #PWR0111
-U 1 1 5F92CDA3
-P 10350 3650
-F 0 "#PWR0111" H 10350 3750 50  0001 C CNN
-F 1 "-12V" H 10365 3823 50  0000 C CNN
-F 2 "" H 10350 3650 50  0001 C CNN
-F 3 "" H 10350 3650 50  0001 C CNN
-	1    10350 3650
-	1    0    0    -1
-$EndComp
-Wire Wire Line
-	10350 3650 10350 4050
-Wire Wire Line
-	8850 3300 8850 4600
-Wire Wire Line
-	8750 4050 10350 4050
-Connection ~ 8750 4050
-Wire Wire Line
-	8750 4050 8750 4600
+Wire Wire Line
+	9550 4600 9550 4400
+Wire Wire Line
+	9550 4400 8450 4400
 $EndSCHEMATC
